Commit message: 2/23

File: catkin_ws/src/mars_robot/description/lidar.xacro (robot description, xacro)
@@ -1,10 +1,10 @@
 <?xml version="1.0"?>
 <robot xmlns:xacro="http://www.ros.org/wiki/xacro" >
-    <joint name="laser_joint" type="fixed">
+    <joint name="laser" type="fixed">
         <parent link="chassis"/>
-        <child link="laser_frame"/>
-        <origin xyz=".90 0 0.25" rpy="0 0 0"/>
+        <child link="laser"/>
+        <origin xyz=".35 0 0.05" rpy="0 0 0"/>
     </joint>
-    <link name="laser_frame">
+    <link name="laser">
         <visual>
             <geometry>
@@ -22,5 +22,5 @@
         </xacro:inertial_cylinder>
     </link>
-    <gazebo reference="laser_frame">
+    <gazebo reference="laser">
         <material>Gazebo/Red</material>
         <sensor name="laser" type="gpu_ray">

Commit message: Updated Robot Model

File: catkin_ws/src/mars_robot/description/lidar.xacro (robot description, xacro)
@@ -1,8 +1,29 @@
 <?xml version="1.0"?>
 <robot xmlns:xacro="http://www.ros.org/wiki/xacro" >
+    <joint name="laser_arm_joint" type="fixed">
+        <parent link="chassis"/>
+        <child link="laser_arm"/>
+        <origin xyz=".90 0 0.25" rpy="0 0 0"/>
+    </joint>
+    <link name="laser_arm">
+        <visual>
+            <geometry>
+                <box size=".2 .2 0.1"/>
+            </geometry>
+            <material name="white"/>
+        </visual>
+        <collision>
+            <geometry>
+                <box size=".2 .2 0.1"/>
+            </geometry>
+        </collision>
+        <xacro:inertial_box mass="2" x=".2" y=".2" z=".1">
+            <origin xyz="0 0 0" rpy="0 0 0"/>
+        </xacro:inertial_box>
+    </link>
     <joint name="laser" type="fixed">
-        <parent link="chassis"/>
+        <parent link="laser_arm"/>
         <child link="laser"/>
-        <origin xyz=".35 0 0.05" rpy="0 0 0"/>
+        <origin xyz=".05 0 -0.07" rpy="0 0 0"/>
     </joint>
     <link name="laser">
@@ -11,5 +32,5 @@
                 <cylinder radius="0.05" length="0.04"/>
             </geometry>
-            <material name="red"/>
+            <material name="blue"/>
         </visual>
         <collision>

File: catkin_ws/src/mars_robot/description/rover_core.xacro (robot description, xacro)
@@ -25,182 +25,177 @@
         <parent link="base_link"/>
         <child link="chassis"/>
-        <origin xyz="-0.1 0 0"/>
+        <origin xyz="-0.1 0 0.1"/>
     </joint>
     <link name="chassis">
         <visual>
+            <origin xyz=".5 0 .2"/>
+            <geometry>
+                <box size=".75 .5 0.35"/>
+            </geometry>
+            <material name="white"/>
+        </visual>
+        <collision>
             <origin xyz=".5 0 .25"/>
             <geometry>
-                <box size=".75 .6 0.5"/>
-            </geometry>
-            <material name="white"/>
-        </visual>
-        <collision>
-            <origin xyz=".5 0 .25"/>
-            <geometry>
-                <box size=".75 .6 0.5"/>
-            </geometry>
-        </collision>
-        <xacro:inertial_box mass="42" x="1" y="1" z=".5">
+                <box size=".75 .5 0.35"/>
+            </geometry>
+        </collision>
+        <xacro:inertial_box mass="42" x="1" y="1" z=".4">
+            <origin xyz=".5 0 .2" rpy="0 0 0"/>
+        </xacro:inertial_box>
+    </link>
+    <gazebo reference="chassis">
+        <material>Gazebo/White</material>
+    </gazebo>
+ <!-- LEFT DRIVE WHEEL 1 LINK -->
+    <joint name="left_drive_wheel_1_joint" type="fixed">
+        <parent link="base_link"/>
+        <child link="left_drive_wheel_1_train"/>
+        <origin xyz=".15 -.25 .1" rpy="${pi/2} 0 0"/>
+        <axis xyz="0 0 1"/>
+    </joint>
+    <link name="left_drive_wheel_1_train">
+        <visual>
+            <geometry>
+                <cylinder radius=".1" length=".08"/>
+            </geometry>
+            <material name="black"/>
+        </visual>
+        <collision>
+            <geometry>
+                <cylinder radius=".1" length=".08"/>
+            </geometry>
+        </collision>
+        <xacro:inertial_cylinder mass="3" length=".08" radius=".1">
+            <origin xyz="0 0 0" rpy="0 0 0"/>
+        </xacro:inertial_cylinder>
+    </link>
+ <!-- LEFT DRIVE WHEEL 3 LINK -->
+    <gazebo reference="left_drive_wheel_1_train">
+        <material>Gazebo/Black</material>
+    </gazebo>
+    <joint name="left_drive_wheel_3_joint" type="fixed">
+        <parent link="base_link"/>
+        <child link="left_drive_wheel_3_train"/>
+        <origin xyz=".6 -.25 .1" rpy="${pi/2} 0 0"/>
+        <axis xyz="0 0 1"/>
+    </joint>
+    <link name="left_drive_wheel_3_train">
+        <visual>
+            <geometry>
+                <cylinder radius=".1" length=".08"/>
+            </geometry>
+            <material name="black"/>
+        </visual>
+        <collision>
+            <geometry>
+                <cylinder radius=".1" length=".08"/>
+            </geometry>
+        </collision>
+        <xacro:inertial_cylinder mass="3" length=".08" radius=".1">
+            <origin xyz="0 0 0" rpy="0 0 0"/>
+        </xacro:inertial_cylinder>
+    </link>
+    <gazebo reference="left_drive_wheel_3_train">
+        <material>Gazebo/Black</material>
+    </gazebo>
+<!-- RIGHT DRIVE WHEEL 1 LINK -->
+    <joint name="right_drive_wheel_1_joint" type="fixed">
+        <parent link="base_link"/>
+        <child link="right_drive_wheel_1_train"/>
+        <origin xyz=".15 .25 .1" rpy="-${pi/2} 0 0"/>
+        <axis xyz="0 0 -1"/>
+    </joint>
+    <link name="right_drive_wheel_1_train">
+        <visual>
+            <geometry>
+                <cylinder radius=".1" length=".08"/>
+            </geometry>
+            <material name="black"/>
+        </visual>
+        <collision>
+            <geometry>
+                <cylinder radius=".1" length=".08"/>
+            </geometry>
+        </collision>
+        <xacro:inertial_cylinder mass="3" length=".08" radius=".1">
+            <origin xyz="0 0 0" rpy="0 0 0"/>
+        </xacro:inertial_cylinder>
+    </link>
+    <gazebo reference="right_drive_wheel_1_train">
+        <material>Gazebo/Black</material>
+    </gazebo>
+<!-- RIGHT DRIVE WHEEL 3 LINK -->
+    <joint name="right_drive_wheel_3_joint" type="fixed">
+        <parent link="base_link"/>
+        <child link="right_drive_wheel_3_train"/>
+        <origin xyz=".6 .25 .1" rpy="-${pi/2} 0 0"/>
+        <axis xyz="0 0 -1"/>
+    </joint>
+    <link name="right_drive_wheel_3_train">
+        <visual>
+            <geometry>
+                <cylinder radius=".1" length=".08"/>
+            </geometry>
+            <material name="black"/>
+        </visual>
+        <collision>
+            <geometry>
+                <cylinder radius=".1" length=".08"/>
+            </geometry>
+        </collision>
+        <xacro:inertial_cylinder mass="3" length=".08" radius=".1">
+            <origin xyz="0 0 0" rpy="0 0 0"/>
+        </xacro:inertial_cylinder>
+    </link>
+    <gazebo reference="right_drive_wheel_3_train">
+        <material>Gazebo/Black</material>
+    </gazebo>
+<!-- RIGHT TREDS -->
+    <joint name="right_tread_joint" type="fixed">
+        <parent link="base_link"/>
+        <child link="right_tred"/>
+        <origin xyz=".375 .25 .1"/>
+    </joint>
+    <link name="right_tred">
+        <visual>
+            <geometry>
+                <box size=".45 .08 0.2"/>
+            </geometry>
+            <material name="black"/>
+        </visual>
+        <collision>
+            <geometry>
+                <box size=".45 .08 0.2"/>
+            </geometry>
+        </collision>
+        <xacro:inertial_box mass="2" x=".45" y=".08" z=".3">
             <origin xyz=".5 0 .25" rpy="0 0 0"/>
         </xacro:inertial_box>
     </link>
-    <gazebo reference="chassis">
-        <material>Gazebo/White</material>
-    </gazebo>
-    <!-- LEFT DRIVE WHEEL 1 LINK -->
-    <joint name="left_drive_wheel_1_joint" type="continuous">
-        <parent link="base_link"/>
-        <child link="left_drive_wheel_1_train"/>
-        <origin xyz=".15 -.3 0" rpy="${pi/2} 0 0"/>
-        <axis xyz="0 0 1"/>
-    </joint>
-    <link name="left_drive_wheel_1_train">
-        <visual>
-            <geometry>
-                <cylinder radius=".15" length=".2"/>
-            </geometry>
-            <material name="black"/>
-        </visual>
-        <collision>
-            <geometry>
-                <cylinder radius=".15" length=".2"/>
-            </geometry>
-        </collision>
-        <xacro:inertial_cylinder mass="3" length=".2" radius=".15">
-            <origin xyz="0 0 0" rpy="0 0 0"/>
-        </xacro:inertial_cylinder>
-    </link>
-    <gazebo reference="left_drive_wheel_1_train">
-        <material>Gazebo/Black</material>
-    </gazebo>
-    <!-- LEFT DRIVE WHEEL 2 LINK -->
-    <!--joint name="left_drive_wheel_2_joint" type="continuous">
-        <parent link="base_link"/>
-        <child link="left_drive_wheel_2_train"/>
-        <origin xyz=".35 -.5 0" rpy="${pi/2} 0 0"/>
-        <axis xyz="0 0 1"/>
-    </joint>
-    <link name="left_drive_wheel_2_train">
-        <visual>
-            <geometry>
-                <cylinder radius=".15" length=".2"/>
-            </geometry>
-            <material name="black"/>
-        </visual>
-        <collision>
-            <geometry>
-                <cylinder radius=".15" length=".2"/>
-            </geometry>
-        </collision>
-        <xacro:inertial_cylinder mass="3" length=".2" radius=".15">
-            <origin xyz="0 0 0" rpy="0 0 0"/>
-        </xacro:inertial_cylinder>
-    </link>
-     <gazebo reference="left_drive_wheel_2_train">
-        <material>Gazebo/Black</material>
-    </gazebo-->
-    <!-- LEFT DRIVE WHEEL 3 LINK -->
-    <joint name="left_drive_wheel_3_joint" type="continuous">
-        <parent link="base_link"/>
-        <child link="left_drive_wheel_3_train"/>
-        <origin xyz=".6 -.3 0" rpy="${pi/2} 0 0"/>
-        <axis xyz="0 0 1"/>
-    </joint>
-    <link name="left_drive_wheel_3_train">
-        <visual>
-            <geometry>
-                <cylinder radius=".15" length=".2"/>
-            </geometry>
-            <material name="black"/>
-        </visual>
-        <collision>
-            <geometry>
-                <cylinder radius=".15" length=".2"/>
-            </geometry>
-        </collision>
-        <xacro:inertial_cylinder mass="3" length=".2" radius=".15">
-            <origin xyz="0 0 0" rpy="0 0 0"/>
-        </xacro:inertial_cylinder>
-    </link>
-    <gazebo reference="left_drive_wheel_3_train">
-        <material>Gazebo/Black</material>
-    </gazebo>
-    <!-- RIGHT DRIVE WHEEL 1 LINK -->
-    <joint name="right_drive_wheel_1_joint" type="continuous">
-        <parent link="base_link"/>
-        <child link="right_drive_wheel_1_train"/>
-        <origin xyz=".15 .3 0" rpy="-${pi/2} 0 0"/>
-        <axis xyz="0 0 -1"/>
-    </joint>
-    <link name="right_drive_wheel_1_train">
-        <visual>
-            <geometry>
-                <cylinder radius=".15" length=".2"/>
-            </geometry>
-            <material name="black"/>
-        </visual>
-        <collision>
-            <geometry>
-                <cylinder radius=".15" length=".2"/>
-            </geometry>
-        </collision>
-        <xacro:inertial_cylinder mass="3" length=".2" radius=".15">
-            <origin xyz="0 0 0" rpy="0 0 0"/>
-        </xacro:inertial_cylinder>
-    </link>
-    <gazebo reference="right_drive_wheel_1_train">
-        <material>Gazebo/Black</material>
-    </gazebo>
-    <!-- RIGHT DRIVE WHEEL 2 LINK -->
-    <!--joint name="right_drive_wheel_2_joint" type="continuous">
-        <parent link="base_link"/>
-        <child link="right_drive_wheel_2_train"/>
-        <origin xyz=".35 .5 0" rpy="-${pi/2} 0 0"/>
-        <axis xyz="0 0 -1"/>
-    </joint>
-    <link name="right_drive_wheel_2_train">
-        <visual>
-            <geometry>
-                <cylinder radius=".15" length=".2"/>
-            </geometry>
-            <material name="black"/>
-        </visual>
-        <collision>
-            <geometry>
-                <cylinder radius=".15" length=".2"/>
-            </geometry>
-        </collision>
-        <xacro:inertial_cylinder mass="3" length=".2" radius=".15">
-            <origin xyz="0 0 0" rpy="0 0 0"/>
-        </xacro:inertial_cylinder>
-    </link>
-    <gazebo reference="right_drive_wheel_2_train">
-        <material>Gazebo/Black</material>
-    </gazebo-->
-    <!-- RIGHT DRIVE WHEEL 3 LINK -->
-    <joint name="right_drive_wheel_3_joint" type="continuous">
-        <parent link="base_link"/>
-        <child link="right_drive_wheel_3_train"/>
-        <origin xyz=".6 .3 0" rpy="-${pi/2} 0 0"/>
-        <axis xyz="0 0 -1"/>
-    </joint>
-    <link name="right_drive_wheel_3_train">
-        <visual>
-            <geometry>
-                <cylinder radius=".15" length=".2"/>
-            </geometry>
-            <material name="black"/>
-        </visual>
-        <collision>
-            <geometry>
-                <cylinder radius=".15" length=".2"/>
-            </geometry>
-        </collision>
-        <xacro:inertial_cylinder mass="3" length=".2" radius=".15">
-            <origin xyz="0 0 0" rpy="0 0 0"/>
-        </xacro:inertial_cylinder>
-    </link>
-    <gazebo reference="right_drive_wheel_3_train">
-        <material>Gazebo/Black</material>
-    </gazebo>
+    <gazebo reference="right_tred">
+        <material>Gazebo/Black</material>
+    </gazebo>
+<!-- LEFT TREDS -->
+    <joint name="left_tread_joint" type="fixed">
+        <parent link="base_link"/>
+        <child link="left_tred"/>
+        <origin xyz=".375 -.25 .1"/>
+    </joint>
+    <link name="left_tred">
+        <visual>
+            <geometry>
+                <box size=".45 .08 0.2"/>
+            </geometry>
+            <material name="black"/>
+        </visual>
+        <collision>
+            <geometry>
+                <box size=".45 .08 0.2"/>
+            </geometry>
+        </collision>
+        <xacro:inertial_box mass="42" x=".45" y=".2" z=".3">
+            <origin xyz=".5 0 .25" rpy="0 0 0"/>
+        </xacro:inertial_box>
+    </link>
 </robot>
